Commit message: update distances from F360

File: Tests/GLaDOS.urdf (robot description, URDF)
Before this commit: robot glados_robot, 5 links, 4 joints
Joints:
- joint head_up_down: origin xyz=0 0 0.059 rpy=0 0 0 -> xyz=0 0 0.083705 rpy=0 0 0
- joint neck_left_right: origin xyz=0 0 0.059 rpy=0 0 0 -> xyz=0 0 0.0641735 rpy=0 0 0
- joint top_to_body: origin xyz=0 0 0.219 rpy=0 0 0 -> xyz=0 0 0.250796 rpy=0 0 0

Commit message: update urdf with better numbers

File: Tests/GLaDOS.urdf (robot description, URDF)
Before this commit: robot glados_robot, 5 links, 4 joints
Links:
- link body_link: geometry visual box size=0.05 0.05 0.05
- link ceiling_link: geometry visual box size=0.01 0.01 0.01
- link head_link: geometry visual box size=0.05 0.05 0.05
- link neck_link: geometry visual box size=0.05 0.05 0.05
Joints:
- joint ceiling_to_top: axis 0 1 0 -> 0 0 1
- joint top_to_body: axis 1 0 0 -> 0 1 0
